File: power-distribution-box/kicad/120.sch (KiCad schematic (older format))
At the start: 13 parts, among them J1 2x5-15R_GFCI, J2 2x5-15R_GFCI, J3 2x5-15R_GFCI, J4 2x5-15R_GFCI, P1 L5-20P, SW1 BREAK, SW2 ENERGIZE, U1 ACA-20PC-4-AC1-RL-C, U2 WA141206GIE

Commit message: 208 bom
Other:
- note added: "EACH BREAKER 5A"
Changed lines of the file:
@@
 Text Notes 600  2200 0    50   ~ 0
 TODO:\nCONSIDER IF L5-30P\nWOULD BE MORE APPROPRIATE
+Text Notes 8150 3250 0    50   ~ 0
+EACH BREAKER 5A
 $EndSCHEMATC
