File: power-distribution-box/kicad/208.sch (KiCad schematic (older format))
At the start: 19 parts, among them J5 L6-20R, J6 L6-20R, P2 L6-30P, SW10 ENABLE, SW3 BREAK, SW4 ENERGIZE, SW5 RESET, SW6 ENABLE, SW7 BREAK, SW8 ENERGIZE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

Commit message: 208 bom
Parts:
- CB5, CB6: value CircuitBreaker_1P -> CircuitBreaker_20A
Changed lines of the file:
@@
 P 2200 4500
 F 0 "CB6" V 1935 4500 50  0000 C CNN
-F 1 "CircuitBreaker_1P" V 2026 4500 50  0000 C CNN
+F 1 "CircuitBreaker_20A" V 2026 4500 50  0000 C CNN
 F 2 "" H 2200 4500 50  0001 C CNN
 F 3 "~" H 2200 4500 50  0001 C CNN
@@
 P 2200 1300
 F 0 "CB5" V 1935 1300 50  0000 C CNN
-F 1 "CircuitBreaker_1P" V 2026 1300 50  0000 C CNN
+F 1 "CircuitBreaker_20A" V 2026 1300 50  0000 C CNN
 F 2 "" H 2200 1300 50  0001 C CNN
 F 3 "~" H 2200 1300 50  0001 C CNN
